Commit message: Updated follower and leader urdf. Deleted unnecessary xacro files

File: turtlebot_ws/src/turtlebot3/turtlebot3_description/urdf/follower.gazebo.xacro (robot description, xacro)
@@ -124,3 +124,45 @@
     </sensor>
   </gazebo>
+  <!--Used wge100_camera info from https://classic.gazebosim.org/tutorials?tut=ros_gzplugins#AddingaSensorPlugin-->
+  <gazebo reference="camera_link">
+    <sensor type="camera" name="camera1">
+      <update_rate>30.0</update_rate>
+      <camera name="head">
+        <horizontal_fov>1.3962634</horizontal_fov>
+        <image>
+          <width>800</width>
+          <height>800</height>
+          <format>R8G8B8</format>
+        </image>
+        <clip>
+          <near>0.02</near>
+          <far>300</far>
+        </clip>
+        <noise>
+          <type>gaussian</type>
+          <!-- Noise is sampled independently per pixel on each frame.
+               That pixel's noise value is added to each of its color
+               channels, which at that point lie in the range [0,1]. -->
+          <mean>0.0</mean>
+          <stddev>0.007</stddev>
+        </noise>
+      </camera>
+      <plugin name="camera_controller" filename="libgazebo_ros_camera.so">
+        <alwaysOn>true</alwaysOn>
+        <updateRate>0.0</updateRate>
+        <cameraName>camera</cameraName>
+        <imageTopicName>image_raw</imageTopicName>
+        <cameraInfoTopicName>camera_info</cameraInfoTopicName>
+        <frameName>camera_link</frameName>
+        <hackBaseline>0.07</hackBaseline>
+        <distortionK1>0.0</distortionK1>
+        <distortionK2>0.0</distortionK2>
+        <distortionK3>0.0</distortionK3>
+        <distortionT1>0.0</distortionT1>
+        <distortionT2>0.0</distortionT2>
+      </plugin>
+    </sensor>
+    <!-- Need this to colour camera in red-->
+    <material>Gazebo/Red</material>
+  </gazebo>
 </robot>

File: turtlebot_ws/src/turtlebot3/turtlebot3_description/urdf/follower.urdf.xacro (robot description, xacro)
@@ -1,35 +1,32 @@
 <?xml version="1.0" ?>
-<robot name="turtlebot3_waffle_pi_for_open_manipulator" xmlns:xacro="http://ros.org/wiki/xacro">
+<robot name="turtlebot3_burger" xmlns:xacro="http://ros.org/wiki/xacro">
   <xacro:include filename="$(find turtlebot3_description)/urdf/common_properties.xacro"/>
-  <xacro:include filename="$(find turtlebot3_description)/urdf/turtlebot3_waffle_pi_for_open_manipulator.gazebo.xacro"/>
+  <xacro:include filename="$(find turtlebot3_description)/urdf/follower.gazebo.xacro"/>
   <link name="base_footprint"/>
   <joint name="base_joint" type="fixed">
     <parent link="base_footprint"/>
-    <child link="base_link" />
-    <origin xyz="0 0 0.010" rpy="0 0 0"/>
+    <child link="base_link"/>
+    <origin xyz="0.0 0.0 0.010" rpy="0 0 0"/>
   </joint>
   <link name="base_link">
     <visual>
-      <origin xyz="-0.064 0 0.0" rpy="0 0 0"/>
+      <origin xyz="-0.032 0 0.0" rpy="0 0 0"/>
       <geometry>
-        <mesh filename="package://turtlebot3_description/meshes/bases/waffle_pi_base_for_open_manipulator.stl" scale="0.001 0.001 0.001"/>
+        <mesh filename="package://turtlebot3_description/meshes/bases/burger_base.stl" scale="0.001 0.001 0.001"/>
       </geometry>
       <material name="light_black"/>
     </visual>
     <collision>
-      <origin xyz="-0.064 0 0.047" rpy="0 0 0"/>
+      <origin xyz="-0.032 0 0.070" rpy="0 0 0"/>
       <geometry>
-        <box size="0.266 0.266 0.094"/>
+        <box size="0.140 0.140 0.143"/>
       </geometry>
     </collision>
     <inertial>
-      <origin xyz="0.0 0 0.0" rpy="0 0 0"/>
-      <mass value="1.6329594e+00"/>
-      <inertia ixx="1.0" ixy="0.0" ixz="0.0"
-               iyy="1.0" iyz="0.0"
-               izz="1.0" />
-      <!-- <inertia ixx="8.7002718e-03" ixy="-4.7576583e-05" ixz="1.1160499e-04"
-               iyy="8.6195418e-03" iyz="-3.5422299e-06"
-               izz="1.4612727e-02" />                -->
+      <origin xyz="0 0 0" rpy="0 0 0"/>
+      <mass value="8.2573504e-01"/>
+      <inertia ixx="2.2124416e-03" ixy="-1.2294101e-05" ixz="3.4938785e-05"
+               iyy="2.1193702e-03" iyz="-5.0120904e-06"
+               izz="2.0064271e-03" />
     </inertial>
   </link>
@@ -37,5 +34,5 @@
     <parent link="base_link"/>
     <child link="wheel_left_link"/>
-    <origin xyz="0.0 0.144 0.023" rpy="-1.57 0 0"/>
+    <origin xyz="0.0 0.08 0.023" rpy="-1.57 0 0"/>
     <axis xyz="0 0 1"/>
   </joint>
@@ -65,5 +62,5 @@
     <parent link="base_link"/>
     <child link="wheel_right_link"/>
-    <origin xyz="0.0 -0.144 0.023" rpy="-1.57 0 0"/>
+    <origin xyz="0.0 -0.080 0.023" rpy="-1.57 0 0"/>
     <axis xyz="0 0 1"/>
   </joint>
@@ -77,5 +74,5 @@
     </visual>
     <collision>
-      <origin xyz="0 0.001 0" rpy="0 0 0"/>
+      <origin xyz="0 0 0" rpy="0 0 0"/>
       <geometry>
         <cylinder length="0.018" radius="0.033"/>
@@ -90,30 +87,10 @@
       </inertial>
   </link>
-  <joint name="caster_back_right_joint" type="fixed">
+  <joint name="caster_back_joint" type="fixed">
     <parent link="base_link"/>
-    <child link="caster_back_right_link"/>
-    <origin xyz="-0.177 -0.064 -0.004" rpy="-1.57 0 0"/>
+    <child link="caster_back_link"/>
+    <origin xyz="-0.081 0 -0.004" rpy="-1.57 0 0"/>
   </joint>
-  <link name="caster_back_right_link">
-    <collision>
-      <origin xyz="0 0.001 0" rpy="0 0 0"/>
-      <geometry>
-        <box size="0.030 0.009 0.020"/>
-      </geometry>
-    </collision>
-    <inertial>
-      <origin xyz="0 0 0" />
-      <mass value="0.005" />
-      <inertia ixx="0.001" ixy="0.0" ixz="0.0"
-               iyy="0.001" iyz="0.0"
-               izz="0.001" />
-    </inertial>
-  </link>
-  <joint name="caster_back_left_joint" type="fixed">
-    <parent link="base_link"/>
-    <child link="caster_back_left_link"/>
-    <origin xyz="-0.177 0.064 -0.004" rpy="-1.57 0 0"/>
-  </joint>
-  <link name="caster_back_left_link">
+  <link name="caster_back_link">
     <collision>
       <origin xyz="0 0.001 0" rpy="0 0 0"/>
@@ -133,5 +110,5 @@
     <parent link="base_link"/>
     <child link="imu_link"/>
-    <origin xyz="0.0 0 0.068" rpy="0 0 0"/>
+    <origin xyz="-0.032 0 0.068" rpy="0 0 0"/>
   </joint>
   <link name="imu_link"/>
@@ -139,5 +116,5 @@
     <parent link="base_link"/>
     <child link="base_scan"/>
-    <origin xyz="-0.024 0 0.122" rpy="0 0 0"/>
+    <origin xyz="-0.032 0 0.172" rpy="0 0 0"/>
   </joint>
   <link name="base_scan">
@@ -152,5 +129,5 @@
       <origin xyz="0.015 0 -0.0065" rpy="0 0 0"/>
       <geometry>
-        <cylinder length="0.0315" radius="0.045"/>
+        <cylinder length="0.0315" radius="0.055"/>
       </geometry>
     </collision>
@@ -163,28 +140,27 @@
     </inertial>
   </link>
+  <!--Creating camera link-->
+  <link name="camera_link">
+    <visual>
+        <geometry>
+            <box size="0.01 0.02 0.01"/>
+        </geometry>
+        <material name="red"/>
+    </visual>
+  </link>
+  <!--Creating camera joint-->
   <joint name="camera_joint" type="fixed">
-    <origin xyz="0.073 -0.011 0.084" rpy="0 0 0"/>
-    <parent link="base_link"/>
+    <parent link="base_footprint"/>
     <child link="camera_link"/>
+    <origin xyz="0.033 0.0 ${0.192/2+0.02}" rpy="0 0 0"/>
   </joint>
-  <link name="camera_link">
-    <collision>
-      <origin xyz="0.005 0.011 0.013" rpy="0 0 0"/>
-      <geometry>
-        <box size="0.015 0.030 0.027"/>
-      </geometry>
-    </collision>
+  <!--Creating camera optical link-->
+  <link name="camera_optical_link">
   </link>
-  <joint name="camera_rgb_joint" type="fixed">
-    <origin xyz="0.003 0.011 0.009" rpy="0 0 0"/>
+  <!--Creating camera optical joint-->
+  <joint name="camera_optical_joint" type="fixed">
     <parent link="camera_link"/>
-    <child link="camera_rgb_frame"/>
+    <child link="camera_optical_link"/>
+    <origin xyz="0.0 0.0 0.0" rpy="${-pi/2} 0 ${-pi/2}"/>
   </joint>
-  <link name="camera_rgb_frame"/>
-  <joint name="camera_rgb_optical_joint" type="fixed">
-    <origin xyz="0 0 0" rpy="-1.57 0 -1.57"/>
-    <parent link="camera_rgb_frame"/>
-    <child link="camera_rgb_optical_frame"/>
-  </joint>
-  <link name="camera_rgb_optical_frame"/>
 </robot>

File: turtlebot_ws/src/turtlebot3/turtlebot3_description/urdf/leader.urdf.xacro (robot description, xacro)
@@ -1,6 +1,7 @@
 <?xml version="1.0" ?>
-<robot name="turtlebot3_burger_for_autorace_2020" xmlns:xacro="http://ros.org/wiki/xacro">
+<robot name="turtlebot3_burger" xmlns:xacro="http://ros.org/wiki/xacro">
   <xacro:include filename="$(find turtlebot3_description)/urdf/common_properties.xacro"/>
-  <xacro:include filename="$(find turtlebot3_description)/urdf/turtlebot3_burger_for_autorace_2020.gazebo.xacro"/>
+  <xacro:include filename="$(find turtlebot3_description)/urdf/leader.gazebo.xacro"/>
+  <xacro:include filename="$(find turtlebot3_description)/urdf/feature.xacro"/>
   <link name="base_footprint"/>
   <joint name="base_joint" type="fixed">
@@ -24,9 +25,9 @@
     </collision>
     <inertial>
-      <origin xyz="-0.016 0 0" rpy="0 0 0"/>
-      <mass value="8.2573504"/>
-      <inertia ixx="2.2124416e-02" ixy="-1.2294101e-04" ixz="3.4938785e-04"
-               iyy="2.1193702e-02" iyz="-5.0120904e-05"
-               izz="2.0064271e-02" />
+      <origin xyz="0 0 0" rpy="0 0 0"/>
+      <mass value="8.2573504e-01"/>
+      <inertia ixx="2.2124416e-03" ixy="-1.2294101e-05" ixz="3.4938785e-05"
+               iyy="2.1193702e-03" iyz="-5.0120904e-06"
+               izz="2.0064271e-03" />
     </inertial>
   </link>
@@ -34,10 +35,10 @@
     <parent link="base_link"/>
     <child link="wheel_left_link"/>
-    <origin xyz="0.0 0.08 0.023" rpy="-1.5707 0 0"/>
+    <origin xyz="0.0 0.08 0.023" rpy="-1.57 0 0"/>
     <axis xyz="0 0 1"/>
   </joint>
   <link name="wheel_left_link">
     <visual>
-      <origin xyz="0 0 0" rpy="1.5707 0 0"/>
+      <origin xyz="0 0 0" rpy="1.57 0 0"/>
       <geometry>
         <mesh filename="package://turtlebot3_description/meshes/wheels/left_tire.stl" scale="0.001 0.001 0.001"/>
@@ -53,8 +54,8 @@
     <inertial>
       <origin xyz="0 0 0" />
-      <mass value="2.8498940" />
-      <inertia ixx="1.1175580e-03" ixy="-4.2369783e-08" ixz="-5.9381719e-07"
-               iyy="1.1192413e-03" iyz="-1.4400107e-08"
-               izz="2.0712558e-03" />
+      <mass value="2.8498940e-02" />
+      <inertia ixx="1.1175580e-05" ixy="-4.2369783e-11" ixz="-5.9381719e-09"
+               iyy="1.1192413e-05" iyz="-1.4400107e-11"
+               izz="2.0712558e-05" />
       </inertial>
   </link>
@@ -62,10 +63,10 @@
     <parent link="base_link"/>
     <child link="wheel_right_link"/>
-    <origin xyz="0.0 -0.080 0.023" rpy="-1.5707 0 0"/>
+    <origin xyz="0.0 -0.080 0.023" rpy="-1.57 0 0"/>
     <axis xyz="0 0 1"/>
   </joint>
   <link name="wheel_right_link">
     <visual>
-      <origin xyz="0 0 0" rpy="1.5707 0 0"/>
+      <origin xyz="0 0 0" rpy="1.57 0 0"/>
       <geometry>
         <mesh filename="package://turtlebot3_description/meshes/wheels/right_tire.stl" scale="0.001 0.001 0.001"/>
@@ -81,8 +82,8 @@
     <inertial>
       <origin xyz="0 0 0" />
-      <mass value="2.8498940" />
-      <inertia ixx="1.1175580e-03" ixy="-4.2369783e-08" ixz="-5.9381719e-07"
-               iyy="1.1192413e-03" iyz="-1.4400107e-08"
-               izz="2.0712558e-03" />
+      <mass value="2.8498940e-02" />
+      <inertia ixx="1.1175580e-05" ixy="-4.2369783e-11" ixz="-5.9381719e-09"
+               iyy="1.1192413e-05" iyz="-1.4400107e-11"
+               izz="2.0712558e-05" />
       </inertial>
   </link>
@@ -90,9 +91,9 @@
     <parent link="base_link"/>
     <child link="caster_back_link"/>
-    <origin xyz="-0.081 0 -0.004" rpy="-1.5707 0 0"/>
+    <origin xyz="-0.081 0 -0.004" rpy="-1.57 0 0"/>
   </joint>
   <link name="caster_back_link">
     <collision>
-      <origin xyz="0 0.000 0" rpy="0 0 0"/>
+      <origin xyz="0 0.001 0" rpy="0 0 0"/>
       <geometry>
         <box size="0.030 0.009 0.020"/>
@@ -101,8 +102,8 @@
     <inertial>
       <origin xyz="0 0 0" />
-      <mass value="0.000001" />
-      <inertia ixx="0.000001" ixy="0.0" ixz="0.0"
-               iyy="0.000001" iyz="0.0"
-               izz="0.000001" />
+      <mass value="0.005" />
+      <inertia ixx="0.001" ixy="0.0" ixz="0.0"
+               iyy="0.001" iyz="0.0"
+               izz="0.001" />
     </inertial>
   </link>
@@ -140,28 +141,3 @@
     </inertial>
   </link>
-  <joint name="camera_dummy_joint" type="fixed">
-    <origin xyz="0.040 -0.000 0.110" rpy="0 0 0"/>
-    <parent link="base_link"/>
-    <child link="camera_dummy_link"/>
-  </joint>
-  <link name="camera_dummy_link">
-    <collision>
-      <origin xyz="0.005 0.000 0.013" rpy="0 0 0"/>
-      <geometry>
-        <box size="0.015 0.030 0.027"/>
-      </geometry>
-    </collision>
-  </link>
-  <joint name="camera_joint" type="fixed">
-    <origin xyz="0.003 0.000 0.009" rpy="0 0 0"/>
-    <parent link="camera_dummy_link"/>
-    <child link="camera_frame"/>
-  </joint>
-  <link name="camera_frame"/>
-  <joint name="camera_optical_joint" type="fixed">
-    <origin xyz="0 0 0" rpy="-1.5707 0 -1.57"/>
-    <parent link="camera_frame"/>
-    <child link="camera_optical_frame"/>
-  </joint>
-  <link name="camera_optical_frame"/>
 </robot>
