Commit message: Modified enviro.launch and feature.xacro to launch different environments. See readme for more details

File: turtlebot_ws/src/turtlebot3/turtlebot3_description/urdf/feature.xacro (robot description, xacro)
@@ -1,19 +1,48 @@
 <?xml version="1.0" ?>
 <robot xmlns:xacro="http://ros.org/wiki/xacro">
+  <!--launch options-->
+  <!--NOTE: By default, environment will run with cylinder-type marker (white)-->
+  <xacro:arg name="use_rectangle" default="false" />
+  <xacro:arg name="marker_blue" default="false" />
   <joint name="feature_joint" type="fixed">
     <parent link="base_footprint"/>
     <child link="feature_link"/>
-    <!--origin xyz="-0.105 0.0 ${0.192/2+0.02}" rpy="0 0 0"/--> <!--Origin for rectangle geometry-->
-    <origin xyz="-0.105 0.0 ${0.192/2+0.02}" rpy="0 ${pi/2} 0"/> <!--Origin for cylinder geometry-->
+    <xacro:if value="$(arg use_rectangle)">
+      <!--Origin for rectangle geometry-->
+      <origin xyz="-0.105 0.0 ${0.192/2+0.02}" rpy="0 0 0" />
+    </xacro:if>
+    <xacro:unless value="$(arg use_rectangle)">
+    <!--Origin for cylinder geometry-->
+    <origin xyz="-0.105 0.0 ${0.192/2+0.02}" rpy="0 ${pi/2} 0"/>
+    </xacro:unless>
   </joint>
   <link name="feature_link">
     <visual>
         <geometry>
-            <!--box size="0.001 0.1 0.1"/--> <!-- Rectangle -->
-            <cylinder radius="0.10" length="0.005"/> <!-- Cylinder -->
+            <xacro:if value="$(arg use_rectangle)">
+              <!-- Rectangle -->
+              <box size="0.001 0.1 0.1"/>
+            </xacro:if>
+            <xacro:unless value="$(arg use_rectangle)">
+            <!-- Cylinder -->
+            <cylinder radius="0.10" length="0.005"/>
+            </xacro:unless>
         </geometry>
-        <material name="white"/>
+        <xacro:if value="$(arg marker_blue)">
+          <material name="blue"/>
+        </xacro:if>
+        <xacro:unless value="$(arg marker_blue)">
+          <material name="white"/>
+        </xacro:unless>
     </visual>
   </link>
+  <!-- GAZEBO -->
+  <gazebo reference="feature_link">
+    <xacro:if value="$(arg marker_blue)">
+      <material>Gazebo/Blue</material>
+    </xacro:if>
+    <xacro:unless value="$(arg marker_blue)">
+      <material>Gazebo/White</material>
+    </xacro:unless>
+  </gazebo>
 </robot>
-<!-- GAZEBO ATTEMPT - not required? -->

Commit message: Updated feature.xacro

File: turtlebot_ws/src/turtlebot3/turtlebot3_description/urdf/feature.xacro (robot description, xacro)
@@ -3,5 +3,5 @@
   <!--launch options-->
   <!--NOTE: By default, environment will run with cylinder-type marker (white)-->
-  <xacro:arg name="use_rectangle" default="false" />
+  <xacro:arg name="use_rectangle" default="true" />
   <xacro:arg name="marker_blue" default="false" />
   <joint name="feature_joint" type="fixed">
@@ -10,9 +10,9 @@
     <xacro:if value="$(arg use_rectangle)">
       <!--Origin for rectangle geometry-->
-      <origin xyz="-0.105 0.0 ${0.192/2+0.02}" rpy="0 0 0" />
+      <origin xyz="0 0.0 0.068" rpy="0 0 0" />
     </xacro:if>
     <xacro:unless value="$(arg use_rectangle)">
     <!--Origin for cylinder geometry-->
-    <origin xyz="-0.105 0.0 ${0.192/2+0.02}" rpy="0 ${pi/2} 0"/>
+    <origin xyz="0 0.0 0.068" rpy="0 ${pi/2} 0"/>
     </xacro:unless>
   </joint>
@@ -22,9 +22,9 @@
             <xacro:if value="$(arg use_rectangle)">
               <!-- Rectangle -->
-              <box size="0.001 0.1 0.1"/>
+              <box size="0.001 0.08 0.08"/>
             </xacro:if>
             <xacro:unless value="$(arg use_rectangle)">
             <!-- Cylinder -->
-            <cylinder radius="0.10" length="0.005"/>
+            <cylinder radius="0.08" length="0.005"/>
             </xacro:unless>
         </geometry>

Commit message: repositioned feature to be behind the lidar

File: turtlebot_ws/src/turtlebot3/turtlebot3_description/urdf/feature.xacro (robot description, xacro)
@@ -10,9 +10,9 @@
     <xacro:if value="$(arg use_rectangle)">
       <!--Origin for rectangle geometry-->
-      <origin xyz="0 0.0 0.068" rpy="0 0 0" />
+      <origin xyz="-0.0965 0.0 0.141" rpy="0 0 0" />
     </xacro:if>
     <xacro:unless value="$(arg use_rectangle)">
     <!--Origin for cylinder geometry-->
-    <origin xyz="0 0.0 0.068" rpy="0 ${pi/2} 0"/>
+    <origin xyz="-0.0965 0.0 0.141" rpy="0 ${pi/2} 0"/>
     </xacro:unless>
   </joint>
